File: minimouse.kicad_pcb (KiCad board)
At the start: 2 copper layers, 90 x 85 mm, 22 parts, among them J1 Conn_ARM_JTAG_SWD_10, J5 Conn_01x02, M1 N20_encoder, M2 N20_encoder, U1 STM32F030C8Tx, U4 HC-SR04

Commit message: tp4
Parts:
- added C10: 22nf, Capacitor_SMD:C_0603_1608Metric, F.Cu at (231.5, 99.0)
- added C11: 22nf, Capacitor_SMD:C_0603_1608Metric, F.Cu at (231.5, 101.5)
- added C12: 2.2µf, Capacitor_SMD:C_0603_1608Metric, F.Cu at (225.4, 96.5)
- added C13: 2.2µf, Capacitor_SMD:C_0603_1608Metric, F.Cu at (214.8, 96.5)
- added C14: 2.2µf, Capacitor_SMD:C_0603_1608Metric, F.Cu at (251.4, 96.5)
- added C15: C, Capacitor_SMD:C_0603_1608Metric, F.Cu at (184.8, 67.0)
- added C7: 2.2µF, Capacitor_SMD:C_0603_1608Metric, F.Cu at (246.8, 110.8)
- added C8: 2.2µF, Capacitor_SMD:C_0603_1608Metric, F.Cu at (246.8, 113.3)
- added C9: 1nf, Capacitor_SMD:C_0603_1608Metric, F.Cu at (231.5, 96.5)
- added D1: LED, LED_SMD:LED_0603_1608Metric, F.Cu at (255.9, 115.2)
- added J2: Conn_01x04, Connector_PinHeader_2.54mm:PinHeader_1x04_P2.54mm_Vertical, F.Cu at (247.1, 97.6)
- added J8: Conn_01x06, Connector_PinHeader_2.54mm:PinHeader_1x06_P2.54mm_Vertical, F.Cu at (122.6, 95.2)
- added J9: Conn_01x06, Connector_PinHeader_2.54mm:PinHeader_1x06_P2.54mm_Vertical, F.Cu at (210.5, 97.6)
- added R10: 10K, Resistor_SMD:R_0603_1608Metric, F.Cu at (137.3, 87.3)
- added R11: 10k, Resistor_SMD:R_0603_1608Metric, F.Cu at (231.5, 106.5)
- added R12: 330, Resistor_SMD:R_0603_1608Metric, F.Cu at (246.8, 115.8)
- added R13: 10K, Resistor_SMD:R_0603_1608Metric, F.Cu at (235.5, 96.5)
- added R14: 1K, Resistor_SMD:R_0603_1608Metric, F.Cu at (235.5, 99.0)
- added R15: 47K, Resistor_SMD:R_0603_1608Metric, F.Cu at (235.5, 101.5)
- added R16: 330m, Resistor_SMD:R_0603_1608Metric, F.Cu at (235.5, 104.0)
- added R17: 330m, Resistor_SMD:R_0603_1608Metric, F.Cu at (235.5, 106.5)
- added R18: 100, Resistor_SMD:R_0603_1608Metric, F.Cu at (225.4, 99.0)
- added R19: 100, Resistor_SMD:R_0603_1608Metric, F.Cu at (214.8, 99.0)
- added R20: 100, Resistor_SMD:R_0603_1608Metric, F.Cu at (225.4, 101.5)
- added R21: 100, Resistor_SMD:R_0603_1608Metric, F.Cu at (214.8, 101.5)
- added R22: R, Resistor_SMD:R_0603_1608Metric, F.Cu at (251.4, 99.0)
- added R23: 100, Resistor_SMD:R_0603_1608Metric, F.Cu at (210.1, 92.0)
- added U2: LP5907MFX-1.2, Package_TO_SOT_SMD:SOT-23-5, F.Cu at (255.5, 109.2)
- added U3: STSPIN240, Package_DFN_QFN:VQFN-16-1EP_3x3mm_P0.5mm_EP1.8x1.8mm, F.Cu at (149.9, 110.0)
- added U4: HC-SR04, minimouse:HC-SR04, F.Cu at (150.0, 69.1)
- moved C5 3.90 mm to (123.2, 86.0)
Connections:
- U1 pad 43: /mcu/UART1_RX -> /external_uart/EXT_UART_TX

Commit message: TP3
Parts:
- moved J9 34.4 mm to (176.6, 91.6)
Changed lines of the file:
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@@
   )
   (footprint "Connector_PinHeader_2.54mm:PinHeader_1x06_P2.54mm_Vertical" (layer "F.Cu")
-    (at 210.4525 97.57)
+    (at 176.6 91.64)
     (descr "Through hole straight pin header, 1x06, 2.54mm pitch, single row")
     (tags "Through hole pin header THT 1x06 2.54mm single row")
