File: mm_motor.kicad_sch (KiCad schematic)
At the start: 1 part, among them M1 N20_encoder

Commit message: tp2
Parts:
- added J2: Conn_01x06_Pin, symbol Connector:Conn_01x06_Pin
Other:
- moved on the sheet: M1
Changed lines of the file:
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@@
 (kicad_sch (version 20230121) (generator eeschema)
   (paper "A4")
+  (wire (pts (xy 118.11 93.98) (xy 118.11 92.71))
+    (stroke (width 0) (type default))
+  )
+  (wire (pts (xy 118.11 96.52) (xy 129.54 96.52))
+    (stroke (width 0) (type default))
+  )
+  (wire (pts (xy 118.11 91.44) (xy 118.11 90.17))
+    (stroke (width 0) (type default))
+  )
+  (wire (pts (xy 118.11 92.71) (xy 130.81 92.71))
+    (stroke (width 0) (type default))
+  )
+  (wire (pts (xy 118.11 99.06) (xy 118.11 96.52))
+    (stroke (width 0) (type default))
+  )
+  (wire (pts (xy 114.3 86.36) (xy 114.3 85.09))
+    (stroke (width 0) (type default))
+  )
+  (wire (pts (xy 129.54 95.25) (xy 129.54 96.52))
+    (stroke (width 0) (type default))
+  )
+  (wire (pts (xy 114.3 85.09) (xy 130.81 85.09))
+    (stroke (width 0) (type default))
+  )
+  (wire (pts (xy 118.11 90.17) (xy 130.81 90.17))
+    (stroke (width 0) (type default))
+  )
   (hierarchical_label "C1" (shape output) (at 118.11 91.44 180) (fields_autoplaced)
     (effects (font (size 1.27 1.27)) (justify right))
@@
     (effects (font (size 1.27 1.27)) (justify right))
   )
-  (hierarchical_label "MA" (shape passive) (at 118.11 86.36 180) (fields_autoplaced)
-    (effects (font (size 1.27 1.27)) (justify right))
+  (hierarchical_label "MA" (shape passive) (at 114.3 86.36 0) (fields_autoplaced)
+    (effects (font (size 1.27 1.27)) (justify left))
   )
-  (symbol (lib_id "minimouse:N20_w_encoder") (at 115.57 57.15 0) (unit 1)
+  (symbol (lib_id "minimouse:N20_w_encoder") (at 110.49 68.58 0) (unit 1)
     (in_bom yes) (on_board yes) (dnp no) (fields_autoplaced)
-    (property "Reference" "M1" (at 118.11 55.88 0)
+    (property "Reference" "M1" (at 113.03 67.31 0)
       (effects (font (size 1.27 1.27)) (justify left))
     )
-    (property "Value" "N20_encoder" (at 118.11 58.42 0)
+    (property "Value" "N20_encoder" (at 113.03 69.85 0)
       (effects (font (size 1.27 1.27)) (justify left))
     )
-    (property "Footprint" "minimouse:N20_with_encoder" (at 118.11 53.34 0)
+    (property "Footprint" "minimouse:N20_with_encoder" (at 113.03 64.77 0)
       (effects (font (size 1.27 1.27)) hide)
     )
-    (property "Datasheet" "" (at 115.57 57.15 0)
+    (property "Datasheet" "" (at 110.49 68.58 0)
       (effects (font (size 1.27 1.27)) hide)
     )
@@
         )
       )
+    )
+  )
+  (symbol (lib_id "Connector:Conn_01x06_Pin") (at 129.54 90.17 0) (unit 1)
+    (in_bom yes) (on_board yes) (dnp no) (fields_autoplaced)
+    (property "Reference" "J2" (at 130.175 80.01 0)
+      (effects (font (size 1.27 1.27)))
+    )
+    (property "Value" "Conn_01x06_Pin" (at 130.175 82.55 0)
+      (effects (font (size 1.27 1.27)))
+    )
+    (property "Footprint" "" (at 129.54 90.17 0)
+      (effects (font (size 1.27 1.27)) hide)
+    )
+    (property "Datasheet" "~" (at 129.54 90.17 0)
+      (effects (font (size 1.27 1.27)) hide)
+    )
+    (pin "3")
+    (pin "4")
+    (pin "5")
+    (pin "2")
+    (pin "6")
+    (pin "1")
+    (instances
+      (project "minimouse"
+        (path "/d8fa4cba-2469-4231-847f-065b6b829f44/7f113667-692a-4f4d-b16f-621d32f3f136"
+          (reference "J2") (unit 1)
+        )
+        (path "/d8fa4cba-2469-4231-847f-065b6b829f44/3975acd0-18ad-47bc-9ce1-d8c4d864aafe"
+          (reference "J3") (unit 1)
+        )
+      )

Commit message: TP3
Parts:
- removed J2: Conn_01x06_Pin, symbol Connector:Conn_01x06_Pin
- added C12: 2.2µf, Capacitor_SMD:C_0603_1608Metric, symbol Device:C
- added J8: Conn_01x06, Connector_PinHeader_2.54mm:PinHeader_1x06_P2.54mm_Vertical, symbol Connector_Generic:Conn_01x06
- added R18, R20: 100, Resistor_SMD:R_0603_1608Metric, symbol Device:R
Connections:
- net C1: now also R18.1
- net C2: now also R20.1
- net MB: now also J8.6 (Pin_6)
- new net: J8.4 (Pin_4), R20.2
- new net: J8.3 (Pin_3), R18.2
- new net +BATT: C12.1, J8.5 (Pin_5)
- new net GND: C12.2
