File: mm_motor_control.kicad_sch (KiCad schematic)
At the start: 0 parts

Commit message: tp2
Parts:
- added C10, C11, C12, C13, C9: C, symbol Device:C
- added R10, R11: R, symbol Device:R
- added Rsensea, Rsenseb: 1k, symbol Device:R
- added U3: STSPIN240, Package_DFN_QFN:VQFN-16-1EP_3x3mm_P0.5mm_EP1.8x1.8mm, symbol Driver_Motor:STSPIN240
Connections:
- net OUT_A1: now also U3.3 (OUTA1)
- net OUT_A2: now also U3.5 (OUTA2)
- net OUT_B1: now also U3.10 (OUTB1)
- net OUT_B2: now also U3.8 (OUTB2)
- net PHASE_A: now also C10.2, U3.1 (PHA)
- net PHASE_B: now also U3.15 (PHB)
- net PWM_A: now also U3.2 (PWMA)
- net PWM_B: now also U3.16 (PWMB)
- net STBY/RESET: now also U3.14 (STBY/RESET)
- new net: R10.2, R11.1, U3.11 (REF)
- new net: Rsensea.1, U3.4 (SENSEA)
- new net: Rsenseb.1, U3.9 (SENSEB)
- new net +BATT: R10.1
- new net GND: R11.2, Rsensea.2, Rsenseb.2, U3.7 (GND)

Commit message: TP3
Parts:
- removed C12, C13: C, symbol Device:C
- removed Rsensea, Rsenseb: 1k, symbol Device:R
- added R13: 10K, Resistor_SMD:R_0603_1608Metric, symbol Device:R
- added R14: 1K, Resistor_SMD:R_0603_1608Metric, symbol Device:R
- added R15: 47K, Resistor_SMD:R_0603_1608Metric, symbol Device:R
- added R16, R17: 330m, Resistor_SMD:R_0603_1608Metric, symbol Device:R
- C10, C11: value C -> 22nf; footprint (none) -> Capacitor_SMD:C_0603_1608Metric
- C9: value C -> 1nf; footprint (none) -> Capacitor_SMD:C_0603_1608Metric
- R10: value R -> 10K; footprint (none) -> Resistor_SMD:R_0603_1608Metric
- R11: value R -> 10k; footprint (none) -> Resistor_SMD:R_0603_1608Metric
Connections:
- net +BATT: now also C11.1, R11.1, U3.6 (VS); no longer R10.1
- net FAULT: now also C9.1, R10.2, U3.13 (EN/FLT)
- net GND: now also C10.2, C11.2, C9.2, U3.17 (EPAD), R13.2, R15.2, R16.1, R17.2; no longer R11.2
- net PHASE_A: no longer C10.2
- net at C10.1: now also R14.2
- net at U3.12 (TOFF): now also R14.1, R15.1
- net at U3.4 (SENSEA): now also R17.1
- net at U3.9 (SENSEB): now also R16.2
- new net: R11.2, R13.1, U3.11 (REF)
