File: mm_power.kicad_sch (KiCad schematic)
At the start: 1 part, among them J5 Conn_01x02

Commit message: tp2
Parts:
- added C7, C8: 1µF, symbol Device:C
- added U2: LP5907MFX-1.2, Package_TO_SOT_SMD:SOT-23-5, symbol Regulator_Linear:LP5907MFX-1.2
Connections:
- net GND: now also U2.2 (GND)
- new net: C7.2, U2.1 (IN)
- new net: C8.2, U2.5 (OUT)
- new net GND1: C7.1
- new net GND2: C8.1
Changed lines of the file:
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@@
   (junction (at 86.36 82.55) (diameter 0) (color 0 0 0 0)
   )
+  (junction (at 116.84 54.61) (diameter 0) (color 0 0 0 0)
+  )
   (junction (at 86.36 95.25) (diameter 0) (color 0 0 0 0)
   )
@@
     (stroke (width 0) (type default))
   )
+  (wire (pts (xy 116.84 54.61) (xy 116.84 55.88))
+    (stroke (width 0) (type default))
+  )
+  (wire (pts (xy 116.84 54.61) (xy 132.08 54.61))
+    (stroke (width 0) (type default))
+  )
   (wire (pts (xy 95.25 82.55) (xy 86.36 82.55))
     (stroke (width 0) (type default))
@@
     (stroke (width 0) (type default))
   )
+  (wire (pts (xy 116.84 54.61) (xy 86.36 54.61))
+    (stroke (width 0) (type default))
+  )
   (wire (pts (xy 95.25 92.71) (xy 95.25 95.25))
     (stroke (width 0) (type default))
   )
+  (wire (pts (xy 147.32 54.61) (xy 160.02 54.61))
+    (stroke (width 0) (type default))
+  )
   (wire (pts (xy 80.01 87.63) (xy 86.36 87.63))
     (stroke (width 0) (type default))
   )
+  (wire (pts (xy 86.36 54.61) (xy 86.36 73.66))
+    (stroke (width 0) (type default))
+  )
   (wire (pts (xy 86.36 95.25) (xy 86.36 100.33))
     (stroke (width 0) (type default))
@@
     (stroke (width 0) (type default))
   )
+  (wire (pts (xy 160.02 54.61) (xy 160.02 57.15))
+    (stroke (width 0) (type default))
+  )
   (wire (pts (xy 80.01 90.17) (xy 86.36 90.17))
     (stroke (width 0) (type default))
   )
   (symbol (lib_id "power:+BATT") (at 86.36 74.93 0) (unit 1)
-    (in_bom yes) (on_board yes) (dnp no) (fields_autoplaced)
+    (in_bom yes) (on_board yes) (dnp no)
     (property "Reference" "#PWR036" (at 86.36 78.74 0)
       (effects (font (size 1.27 1.27)) hide)
     )
-    (property "Value" "+BATT" (at 86.36 69.85 0)
+    (property "Value" "+BATT" (at 83.82 72.39 0)
       (effects (font (size 1.27 1.27)))
     )
@@
     )
   )
+  (symbol (lib_id "power:GND") (at 139.7 64.77 0) (unit 1)
+    (in_bom yes) (on_board yes) (dnp no) (fields_autoplaced)
+    (property "Reference" "#PWR08" (at 139.7 71.12 0)
+      (effects (font (size 1.27 1.27)) hide)
+    )
+    (property "Value" "GND" (at 139.7 69.85 0)
+      (effects (font (size 1.27 1.27)))
+    )
+    (property "Footprint" "" (at 139.7 64.77 0)
+      (effects (font (size 1.27 1.27)) hide)
+    )
+    (property "Datasheet" "" (at 139.7 64.77 0)
+      (effects (font (size 1.27 1.27)) hide)
+    )
+    (pin "1")
+    (instances
+      (project "minimouse"
+        (path "/d8fa4cba-2469-4231-847f-065b6b829f44/3f9b0845-5778-418c-a7a8-03da2392145e"
+          (reference "#PWR08") (unit 1)
+        )
+      )
+    )
+  )
+  (symbol (lib_id "Regulator_Linear:LP5907MFX-1.2") (at 139.7 57.15 0) (unit 1)
+    (in_bom yes) (on_board yes) (dnp no) (fields_autoplaced)
+    (property "Reference" "U2" (at 139.7 46.99 0)
+      (effects (font (size 1.27 1.27)))
+    )
+    (property "Value" "LP5907MFX-1.2" (at 139.7 49.53 0)
+      (effects (font (size 1.27 1.27)))
+    )
+    (property "Footprint" "Package_TO_SOT_SMD:SOT-23-5" (at 139.7 48.26 0)
+      (effects (font (size 1.27 1.27)) hide)
+    )
+    (property "Datasheet" "http://www.ti.com/lit/ds/symlink/lp5907.pdf" (at 139.7 44.45 0)
+      (effects (font (size 1.27 1.27)) hide)
+    )
+    (pin "5")
+    (pin "1")
+    (pin "3")
+    (pin "4")
+    (pin "2")
+    (instances
+      (project "minimouse"
+        (path "/d8fa4cba-2469-4231-847f-065b6b829f44/3f9b0845-5778-418c-a7a8-03da2392145e"
+          (reference "U2") (unit 1)
+        )
+      )
+    )
+  )
+  (symbol (lib_id "power:GND1") (at 116.84 63.5 0) (unit 1)
+    (in_bom yes) (on_board yes) (dnp no) (fields_autoplaced)
+    (property "Reference" "#PWR09" (at 116.84 69.85 0)
+      (effects (font (size 1.27 1.27)) hide)
+    )
+    (property "Value" "GND1" (at 116.84 68.58 0)
+      (effects (font (size 1.27 1.27)))
+    )
+    (property "Footprint" "" (at 116.84 63.5 0)
+      (effects (font (size 1.27 1.27)) hide)
+    )
+    (property "Datasheet" "" (at 116.84 63.5 0)
+      (effects (font (size 1.27 1.27)) hide)
+    )
+    (pin "1")
+    (instances
+      (project "minimouse"
+        (path "/d8fa4cba-2469-4231-847f-065b6b829f44/3f9b0845-5778-418c-a7a8-03da2392145e"
+          (reference "#PWR09") (unit 1)
+        )
+      )
+    )
+  )
+  (symbol (lib_id "power:GND2") (at 160.02 64.77 0) (unit 1)
+    (in_bom yes) (on_board yes) (dnp no) (fields_autoplaced)
+    (property "Reference" "#PWR010" (at 160.02 71.12 0)
+      (effects (font (size 1.27 1.27)) hide)
+    )
+    (property "Value" "GND2" (at 160.02 69.85 0)
+      (effects (font (size 1.27 1.27)))
+    )
+    (property "Footprint" "" (at 160.02 64.77 0)
+      (effects (font (size 1.27 1.27)) hide)
+    )
+    (property "Datasheet" "" (at 160.02 64.77 0)
+      (effects (font (size 1.27 1.27)) hide)
+    )
+    (pin "1")
+    (instances
+      (project "minimouse"
+        (path "/d8fa4cba-2469-4231-847f-065b6b829f44/3f9b0845-5778-418c-a7a8-03da2392145e"
+          (reference "#PWR010") (unit 1)
+        )
+      )
+    )
+  )
   (symbol (lib_id "Connector_Generic:Conn_01x02") (at 74.93 90.17 180) (unit 1)
     (in_bom yes) (on_board yes) (dnp no) (fields_autoplaced)
@@
         )
       )
+    )
+  )
+  (symbol (lib_id "Device:C") (at 116.84 59.69 0) (mirror x) (unit 1)
+    (in_bom yes) (on_board yes) (dnp no)
+    (property "Reference" "C7" (at 120.65 60.96 0)
+      (effects (font (size 1.27 1.27)) (justify left))
+    )
+    (property "Value" "1µF" (at 120.65 58.42 0)
+      (effects (font (size 1.27 1.27)) (justify left))
+    )
+    (property "Footprint" "" (at 117.8052 55.88 0)
+      (effects (font (size 1.27 1.27)) hide)
+    )
+    (property "Datasheet" "~" (at 116.84 59.69 0)
+      (effects (font (size 1.27 1.27)) hide)
+    )
+    (pin "1")
+    (pin "2")
+    (instances
+      (project "minimouse"
+        (path "/d8fa4cba-2469-4231-847f-065b6b829f44/3f9b0845-5778-418c-a7a8-03da2392145e"
+          (reference "C7") (unit 1)
+        )
+      )
+    )
+  )
+  (symbol (lib_id "Device:C") (at 160.02 60.96 0) (mirror x) (unit 1)
+    (in_bom yes) (on_board yes) (dnp no)
+    (property "Reference" "C8" (at 163.83 62.23 0)
+      (effects (font (size 1.27 1.27)) (justify left))
+    )
+    (property "Value" "1µF" (at 163.83 59.69 0)
+      (effects (font (size 1.27 1.27)) (justify left))
+    )
+    (property "Footprint" "" (at 160.9852 57.15 0)
+      (effects (font (size 1.27 1.27)) hide)
+    )
+    (property "Datasheet" "~" (at 160.02 60.96 0)
+      (effects (font (size 1.27 1.27)) hide)
+    )
+    (pin "1")
+    (pin "2")
+    (instances
+      (project "minimouse"
+        (path "/d8fa4cba-2469-4231-847f-065b6b829f44/3f9b0845-5778-418c-a7a8-03da2392145e"
+          (reference "C8") (unit 1)
+        )
+      )

Commit message: TP3
Parts:
- added D1: LED, LED_SMD:LED_0603_1608Metric, symbol Device:LED
- added R12: 330, Resistor_SMD:R_0603_1608Metric, symbol Device:R
- C7, C8: value 1µF -> 2.2µF; footprint (none) -> Capacitor_SMD:C_0603_1608Metric
Connections:
- net GND1 is gone; now on net GND: C7.1
- net GND2 is gone; now on net GND: C8.1
- net GND: now also D1.1 (K)
- net at C7.2, U2.1 (IN): now also U2.3 (EN)
- net +3.3V: now reaches C8.2, U2.5 (OUT)
- net +3.3V: now also R12.1
- new net: D1.2 (A), R12.2
Changed lines of the file:
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@@
   (junction (at 86.36 82.55) (diameter 0) (color 0 0 0 0)
   )
+  (junction (at 160.02 33.02) (diameter 0) (color 0 0 0 0)
+  )
+  (junction (at 160.02 54.61) (diameter 0) (color 0 0 0 0)
+  )
   (junction (at 116.84 54.61) (diameter 0) (color 0 0 0 0)
   )
+  (junction (at 127 54.61) (diameter 0) (color 0 0 0 0)
+  )
+  (junction (at 139.7 64.77) (diameter 0) (color 0 0 0 0)
+  )
   (junction (at 86.36 95.25) (diameter 0) (color 0 0 0 0)
   )
+  (junction (at 160.02 64.77) (diameter 0) (color 0 0 0 0)
+  )
   (wire (pts (xy 86.36 90.17) (xy 86.36 95.25))
     (stroke (width 0) (type default))
   )
+  (wire (pts (xy 139.7 64.77) (xy 160.02 64.77))
+    (stroke (width 0) (type default))
+  )
   (wire (pts (xy 116.84 54.61) (xy 116.84 55.88))
     (stroke (width 0) (type default))
   )
-  (wire (pts (xy 116.84 54.61) (xy 132.08 54.61))
+  (wire (pts (xy 127 54.61) (xy 132.08 54.61))
+    (stroke (width 0) (type default))
+  )
+  (wire (pts (xy 116.84 54.61) (xy 127 54.61))
     (stroke (width 0) (type default))
   )
@@
     (stroke (width 0) (type default))
   )
+  (wire (pts (xy 139.7 72.39) (xy 139.7 64.77))
+    (stroke (width 0) (type default))
+  )
+  (wire (pts (xy 160.02 33.02) (xy 160.02 54.61))
+    (stroke (width 0) (type default))
+  )
   (wire (pts (xy 116.84 54.61) (xy 86.36 54.61))
     (stroke (width 0) (type default))
   )
+  (wire (pts (xy 116.84 63.5) (xy 139.7 63.5))
+    (stroke (width 0) (type default))
+  )
   (wire (pts (xy 95.25 92.71) (xy 95.25 95.25))
     (stroke (width 0) (type default))
@@
     (stroke (width 0) (type default))
   )
+  (wire (pts (xy 175.26 39.37) (xy 175.26 33.02))
+    (stroke (width 0) (type default))
+  )
+  (wire (pts (xy 160.02 33.02) (xy 175.26 33.02))
+    (stroke (width 0) (type default))
+  )
   (wire (pts (xy 86.36 95.25) (xy 86.36 100.33))
     (stroke (width 0) (type default))
@@
     (stroke (width 0) (type default))
   )
+  (wire (pts (xy 175.26 46.99) (xy 175.26 54.61))
+    (stroke (width 0) (type default))
+  )
   (wire (pts (xy 86.36 82.55) (xy 86.36 87.63))
     (stroke (width 0) (type default))
@@
     (stroke (width 0) (type default))
   )
+  (wire (pts (xy 139.7 63.5) (xy 139.7 64.77))
+    (stroke (width 0) (type default))
+  )
+  (wire (pts (xy 132.08 57.15) (xy 127 57.15))
+    (stroke (width 0) (type default))
+  )
+  (wire (pts (xy 160.02 64.77) (xy 175.26 64.77))
+    (stroke (width 0) (type default))
+  )
   (wire (pts (xy 80.01 90.17) (xy 86.36 90.17))
+    (stroke (width 0) (type default))
+  )
+  (wire (pts (xy 127 54.61) (xy 127 57.15))
+    (stroke (width 0) (type default))
+  )
+  (wire (pts (xy 175.26 62.23) (xy 175.26 64.77))
     (stroke (width 0) (type default))
   )
@@
     )
   )
-  (symbol (lib_id "power:GND") (at 139.7 64.77 0) (unit 1)
-    (in_bom yes) (on_board yes) (dnp no) (fields_autoplaced)
-    (property "Reference" "#PWR08" (at 139.7 71.12 0)
-      (effects (font (size 1.27 1.27)) hide)
-    )
-    (property "Value" "GND" (at 139.7 69.85 0)
-      (effects (font (size 1.27 1.27)))
-    )
-    (property "Footprint" "" (at 139.7 64.77 0)
-      (effects (font (size 1.27 1.27)) hide)
-    )
-    (property "Datasheet" "" (at 139.7 64.77 0)
+  (symbol (lib_id "power:GND") (at 139.7 72.39 0) (unit 1)
+    (in_bom yes) (on_board yes) (dnp no) (fields_autoplaced)
+    (property "Reference" "#PWR08" (at 139.7 78.74 0)
+      (effects (font (size 1.27 1.27)) hide)
+    )
+    (property "Value" "GND" (at 139.7 77.47 0)
+      (effects (font (size 1.27 1.27)))
+    )
+    (property "Footprint" "" (at 139.7 72.39 0)
+      (effects (font (size 1.27 1.27)) hide)
+    )
+    (property "Datasheet" "" (at 139.7 72.39 0)
       (effects (font (size 1.27 1.27)) hide)
     )
@@
         (path "/d8fa4cba-2469-4231-847f-065b6b829f44/3f9b0845-5778-418c-a7a8-03da2392145e"
           (reference "#PWR08") (unit 1)
+        )
+      )
+    )
+  )
+  (symbol (lib_id "Device:R") (at 175.26 43.18 0) (unit 1)
+    (in_bom yes) (on_board yes) (dnp no) (fields_autoplaced)
+    (property "Reference" "R12" (at 177.8 41.91 0)
+      (effects (font (size 1.27 1.27)) (justify left))
+    )
+    (property "Value" "330" (at 177.8 44.45 0)
+      (effects (font (size 1.27 1.27)) (justify left))
+    )
+    (property "Footprint" "Resistor_SMD:R_0603_1608Metric" (at 173.482 43.18 90)
+      (effects (font (size 1.27 1.27)) hide)
+    )
+    (property "Datasheet" "~" (at 175.26 43.18 0)
+      (effects (font (size 1.27 1.27)) hide)
+    )
+    (pin "1")
+    (pin "2")
+    (instances
+      (project "minimouse"
+        (path "/d8fa4cba-2469-4231-847f-065b6b829f44/3f9b0845-5778-418c-a7a8-03da2392145e"
+          (reference "R12") (unit 1)
         )
       )
@@
     )
   )
-  (symbol (lib_id "power:GND1") (at 116.84 63.5 0) (unit 1)
-    (in_bom yes) (on_board yes) (dnp no) (fields_autoplaced)
-    (property "Reference" "#PWR09" (at 116.84 69.85 0)
-      (effects (font (size 1.27 1.27)) hide)
-    )
-    (property "Value" "GND1" (at 116.84 68.58 0)
-      (effects (font (size 1.27 1.27)))
-    )
-    (property "Footprint" "" (at 116.84 63.5 0)
-      (effects (font (size 1.27 1.27)) hide)
-    )
-    (property "Datasheet" "" (at 116.84 63.5 0)
-      (effects (font (size 1.27 1.27)) hide)
-    )
-    (pin "1")
-    (instances
-      (project "minimouse"
-        (path "/d8fa4cba-2469-4231-847f-065b6b829f44/3f9b0845-5778-418c-a7a8-03da2392145e"
-          (reference "#PWR09") (unit 1)
-        )
-      )
-    )
-  )
-  (symbol (lib_id "power:GND2") (at 160.02 64.77 0) (unit 1)
-    (in_bom yes) (on_board yes) (dnp no) (fields_autoplaced)
-    (property "Reference" "#PWR010" (at 160.02 71.12 0)
-      (effects (font (size 1.27 1.27)) hide)
-    )
-    (property "Value" "GND2" (at 160.02 69.85 0)
-      (effects (font (size 1.27 1.27)))
-    )
-    (property "Footprint" "" (at 160.02 64.77 0)
-      (effects (font (size 1.27 1.27)) hide)
-    )
-    (property "Datasheet" "" (at 160.02 64.77 0)
-      (effects (font (size 1.27 1.27)) hide)
-    )
-    (pin "1")
-    (instances
-      (project "minimouse"
-        (path "/d8fa4cba-2469-4231-847f-065b6b829f44/3f9b0845-5778-418c-a7a8-03da2392145e"
-          (reference "#PWR010") (unit 1)
+  (symbol (lib_id "power:+3.3V") (at 160.02 33.02 0) (unit 1)
+    (in_bom yes) (on_board yes) (dnp no) (fields_autoplaced)
+    (property "Reference" "#PWR017" (at 160.02 36.83 0)
+      (effects (font (size 1.27 1.27)) hide)
+    )
+    (property "Value" "+3.3V" (at 160.02 27.94 0)
+      (effects (font (size 1.27 1.27)))
+    )
+    (property "Footprint" "" (at 160.02 33.02 0)
+      (effects (font (size 1.27 1.27)) hide)
+    )
+    (property "Datasheet" "" (at 160.02 33.02 0)
+      (effects (font (size 1.27 1.27)) hide)
+    )
+    (pin "1")
+    (instances
+      (project "minimouse"
+        (path "/d8fa4cba-2469-4231-847f-065b6b829f44/3f9b0845-5778-418c-a7a8-03da2392145e"
+          (reference "#PWR017") (unit 1)
+        )
+      )
+    )
+  )
+  (symbol (lib_id "Device:LED") (at 175.26 58.42 90) (unit 1)
+    (in_bom yes) (on_board yes) (dnp no) (fields_autoplaced)
+    (property "Reference" "D1" (at 179.07 58.7375 90)
+      (effects (font (size 1.27 1.27)) (justify right))
+    )
+    (property "Value" "LED" (at 179.07 61.2775 90)
+      (effects (font (size 1.27 1.27)) (justify right))
+    )
+    (property "Footprint" "LED_SMD:LED_0603_1608Metric" (at 175.26 58.42 0)
+      (effects (font (size 1.27 1.27)) hide)
+    )
+    (property "Datasheet" "~" (at 175.26 58.42 0)
+      (effects (font (size 1.27 1.27)) hide)
+    )
+    (pin "1")
+    (pin "2")
+    (instances
+      (project "minimouse"
+        (path "/d8fa4cba-2469-4231-847f-065b6b829f44/3f9b0845-5778-418c-a7a8-03da2392145e"
+          (reference "D1") (unit 1)
         )
       )
@@
       (effects (font (size 1.27 1.27)) (justify left))
     )
-    (property "Value" "1µF" (at 120.65 58.42 0)
-      (effects (font (size 1.27 1.27)) (justify left))
-    )
-    (property "Footprint" "" (at 117.8052 55.88 0)
+    (property "Value" "2.2µF" (at 120.65 58.42 0)
+      (effects (font (size 1.27 1.27)) (justify left))
+    )
+    (property "Footprint" "Capacitor_SMD:C_0603_1608Metric" (at 117.8052 55.88 0)
       (effects (font (size 1.27 1.27)) hide)
     )
@@
       (effects (font (size 1.27 1.27)) (justify left))
     )
-    (property "Value" "1µF" (at 163.83 59.69 0)
-      (effects (font (size 1.27 1.27)) (justify left))
-    )
-    (property "Footprint" "" (at 160.9852 57.15 0)
-      (effects (font (size 1.27 1.27)) hide)
-    )
+    (property "Value" "2.2µF" (at 163.83 59.69 0)
+      (effects (font (size 1.27 1.27)) (justify left))
+    )
+    (property "Footprint" "Capacitor_SMD:C_0603_1608Metric" (at 160.9852 57.15 0)
+      (effects (font (size 1.27 1.27)) hide)
+    )
